File: touch-pads/touch-pads.kicad_pcb (KiCad board)
At the start: 2 copper layers, 120 x 148.2 mm, 14 parts, among them J1 Conn_01x06_Pin, J2 Conn_01x06_Socket, J3 Conn_01x06_Pin, K1 Conn_01x01, K2 Conn_01x01, K3 Conn_01x01, K4 Conn_01x01, K5 Conn_01x01, K6 Conn_01x01, K7 Conn_01x01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

Commit message: large board
Parts:
- removed J2: Conn_01x06_Socket, Connector_PinSocket_2.54mm:PinSocket_1x06_P2.54mm_Horizontal
- removed J3: Conn_01x06_Pin, Connector_PinHeader_2.54mm:PinHeader_1x06_P2.54mm_Horizontal
- removed R15: 10k, Resistor_SMD:R_0805_2012Metric_Pad1.20x1.40mm_HandSolder
- removed R19: 150k, Resistor_SMD:R_0805_2012Metric_Pad1.20x1.40mm_HandSolder
- removed U8: CAP1188-1-CP-TR, CAP1188_1_CP_TR:QFN24_4X4MC_MCH
- added K10: Conn_01x01, TouchKey:TouchKey_Standard, F.Cu at (193.8, 218.8)
- added K11: Conn_01x01, TouchKey:TouchKey_Standard, F.Cu at (223.8, 164.8)
- added K12: Conn_01x01, TouchKey:TouchKey_Standard, F.Cu at (223.8, 218.8)
- added K13: Conn_01x01, TouchKey:TouchKey_Standard, F.Cu at (253.8, 164.8)
- added K14: Conn_01x01, TouchKey:TouchKey_Standard, F.Cu at (253.8, 218.8)
- added K15: Conn_01x01, TouchKey:TouchKey_Standard, F.Cu at (283.8, 164.8)
- added K16: Conn_01x01, TouchKey:TouchKey_Standard, F.Cu at (283.8, 218.8)
- added K17: Conn_01x01, TouchKey:TouchKey_Standard, F.Cu at (313.8, 164.8)
- added K18: Conn_01x01, TouchKey:TouchKey_Standard, F.Cu at (313.8, 218.8)
- added K19: Conn_01x01, TouchKey:TouchKey_Standard, F.Cu at (343.8, 164.8)
- added K20: Conn_01x01, TouchKey:TouchKey_Standard, F.Cu at (343.8, 218.8)
- added K21: Conn_01x01, TouchKey:TouchKey_Standard, F.Cu at (373.8, 164.8)
- added K22: Conn_01x01, TouchKey:TouchKey_Standard, F.Cu at (373.8, 218.8)
- added K23: Conn_01x01, TouchKey:TouchKey_Standard, F.Cu at (403.8, 164.8)
- added K24: Conn_01x01, TouchKey:TouchKey_Standard, F.Cu at (403.8, 218.8)
- added K25: Conn_01x01, TouchKey:TouchKey_Standard, F.Cu at (433.8, 164.8)
- added K26: Conn_01x01, TouchKey:TouchKey_Standard, F.Cu at (433.8, 218.8)
- added K27: Conn_01x01, TouchKey:TouchKey_Standard, F.Cu at (463.8, 164.8)
- added K28: Conn_01x01, TouchKey:TouchKey_Standard, F.Cu at (463.8, 218.8)
- added K29: Conn_01x01, TouchKey:TouchKey_Standard, F.Cu at (493.8, 164.8)
- added K30: Conn_01x01, TouchKey:TouchKey_Standard, F.Cu at (493.8, 218.8)
- added K31: Conn_01x01, TouchKey:TouchKey_Standard, F.Cu at (523.8, 164.8)
- added K32: Conn_01x01, TouchKey:TouchKey_Standard, F.Cu at (523.8, 218.8)
- added K9: Conn_01x01, TouchKey:TouchKey_Standard, F.Cu at (193.8, 164.8)
- added R1: 10k, Resistor_SMD:R_0805_2012Metric_Pad1.20x1.40mm_HandSolder, F.Cu at (116.2, 258.8)
- added R2: 10k, Resistor_SMD:R_0805_2012Metric_Pad1.20x1.40mm_HandSolder, F.Cu at (356.2, 258.8)
- added R3: 150k, Resistor_SMD:R_0805_2012Metric_Pad1.20x1.40mm_HandSolder, F.Cu at (130.5, 253.0)
- added R4: 100k, Resistor_SMD:R_0805_2012Metric_Pad1.20x1.40mm_HandSolder, F.Cu at (370.5, 253.0)
- added R5: 10k, Resistor_SMD:R_0805_2012Metric_Pad1.20x1.40mm_HandSolder, F.Cu at (250.5, 253.0)
- added R6: 10k, Resistor_SMD:R_0805_2012Metric_Pad1.20x1.40mm_HandSolder, F.Cu at (476.2, 258.8)
- added R7: 120k, Resistor_SMD:R_0805_2012Metric_Pad1.20x1.40mm_HandSolder, F.Cu at (236.2, 258.8)
- added R8: 82k, Resistor_SMD:R_0805_2012Metric_Pad1.20x1.40mm_HandSolder, F.Cu at (490.5, 253.0)
- added U1: CAP1188-1-CP-TR, CAP1188_1_CP_TR:QFN24_4X4MC_MCH, F.Cu at (124.2, 256.7)
- added U2: CAP1188-1-CP-TR, CAP1188_1_CP_TR:QFN24_4X4MC_MCH, F.Cu at (364.2, 256.8)
- added U3: CAP1188-1-CP-TR, CAP1188_1_CP_TR:QFN24_4X4MC_MCH, F.Cu at (244.2, 256.8)
- added U4: CAP1188-1-CP-TR, CAP1188_1_CP_TR:QFN24_4X4MC_MCH, F.Cu at (484.2, 256.8)
- J1: value Conn_01x06_Pin -> Conn_01x06_Socket; footprint Connector_PinHeader_2.54mm:PinHeader_1x06_P2.54mm_Horizontal -> Connector_JST:JST_XH_B6B-XH-A_1x06_P2.50mm_Vertical; moved to B.Cu
- moved J1 326.7 mm to (304.0, 255.5)
- moved K1 73.3 mm to (73.8, 164.8)
- moved K2 73.3 mm to (73.8, 218.8)
- moved K3 73.3 mm to (103.8, 164.8)
- moved K4 73.3 mm to (103.8, 218.8)
- moved K5 73.3 mm to (133.8, 164.8)
- moved K6 73.3 mm to (133.8, 218.8)
- moved K7 73.3 mm to (163.8, 164.8)
- moved K8 73.3 mm to (163.8, 218.8)
Connections:
- J1 pad 1: ALERT -> SMCLK
- J1 pad 2: RESET -> SMDATA
- J1 pad 3: SMDATA -> RESET
- J1 pad 4: SMCLK -> +3.3V
- J1 pad 5: +3.3V -> GND
- J1 pad 6: GND -> ALERT
Routing:
- net GND: track 0.00 -> 468.9 mm, vias 0 -> 4
- net ALERT: track 0.00 -> 377.4 mm, vias 0 -> 4
- net SMCLK: track 0.00 -> 376.5 mm, vias 0 -> 4
- net +3.3V: track 0.00 -> 376.3 mm, vias 0 -> 4
- net RESET: track 0.00 -> 372.5 mm, vias 0 -> 4
- net SMDATA: track 0.00 -> 371.2 mm, vias 0 -> 4
- net Net-(K1-Pin_1): track 0.00 -> 155.3 mm
- net Net-(K9-Pin_1): track 0.00 -> 155.3 mm
- net Net-(K25-Pin_1): track 0.00 -> 155.3 mm
- net Net-(K17-Pin_1): track 0.00 -> 155.3 mm
- net Net-(K3-Pin_1): track 0.00 -> 124.0 mm
- net Net-(K27-Pin_1): track 0.00 -> 124.0 mm
- net Net-(K19-Pin_1): track 0.00 -> 124.0 mm
- net Net-(K11-Pin_1): track 0.00 -> 124.0 mm
- net Net-(K7-Pin_1): track 0.00 -> 118.5 mm
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Other:
- board size 120 x 148.2 mm -> 479.8 x 128.2 mm
- board text added: "K2"
- board text added: "K4"
- board text added: "K7"

Commit message: more work
Parts:
- added REF**: MountingHole_3.2mm_M3, MountingHole:MountingHole_3.2mm_M3, F.Cu at (298.8, 259.0)
- added REF**: MountingHole_3.2mm_M3, MountingHole:MountingHole_3.2mm_M3, F.Cu at (542.8, 132.8)
- added REF**: MountingHole_3.2mm_M3, MountingHole:MountingHole_3.2mm_M3, F.Cu at (418.8, 259.0)
- added REF**: MountingHole_3.2mm_M3, MountingHole:MountingHole_3.2mm_M3, F.Cu at (178.8, 132.8)
- added REF**: MountingHole_3.2mm_M3, MountingHole:MountingHole_3.2mm_M3, F.Cu at (298.8, 132.8)
- added REF**: MountingHole_3.2mm_M3, MountingHole:MountingHole_3.2mm_M3, F.Cu at (542.8, 259.0)
- added REF**: MountingHole_3.2mm_M3, MountingHole:MountingHole_3.2mm_M3, F.Cu at (54.8, 132.8)
- added REF**: MountingHole_3.2mm_M3, MountingHole:MountingHole_3.2mm_M3, F.Cu at (54.8, 259.0)
- added REF**: MountingHole_3.2mm_M3, MountingHole:MountingHole_3.2mm_M3, F.Cu at (418.8, 132.8)
- added REF**: MountingHole_3.2mm_M3, MountingHole:MountingHole_3.2mm_M3, F.Cu at (178.8, 259.0)
- moved J1 22.7 mm to (281.5, 258.5)
- moved R5 15.4 mm to (236.2, 258.8), turned to -90 degrees
- moved R7 15.4 mm to (250.5, 253.0), turned to 0 degrees
Routing:
- net SMDATA: track 371.2 -> 389.2 mm
- net SMCLK: track 376.5 -> 394.6 mm
- net +3.3V: track 376.3 -> 393.3 mm
- net RESET: track 372.5 -> 389.1 mm
- net GND: track 468.9 -> 484.1 mm
- net ALERT: track 377.4 -> 389.6 mm
Other:
- board size 479.8 x 128.2 mm -> 500 x 138.2 mm
- board text removed: "K2"
- board text removed: "K4"
- board text removed: "K7"

Commit message: add bypass caps
Parts:
- added C1: 0.1uF, Capacitor_SMD:C_0805_2012Metric_Pad1.18x1.45mm_HandSolder, F.Cu at (115.2, 258.5)
- added C2: 10uF, Capacitor_SMD:C_0805_2012Metric_Pad1.18x1.45mm_HandSolder, F.Cu at (117.8, 258.5)
- added C3: 0.1uF, Capacitor_SMD:C_0805_2012Metric_Pad1.18x1.45mm_HandSolder, F.Cu at (235.2, 258.7)
- added C4: 10uF, Capacitor_SMD:C_0805_2012Metric_Pad1.18x1.45mm_HandSolder, F.Cu at (237.8, 258.8)
- added C5: 0.1uF, Capacitor_SMD:C_0805_2012Metric_Pad1.18x1.45mm_HandSolder, F.Cu at (355.2, 258.5)
- added C6: 10uF, Capacitor_SMD:C_0805_2012Metric_Pad1.18x1.45mm_HandSolder, F.Cu at (357.8, 258.5)
- added C7: 0.1uF, Capacitor_SMD:C_0805_2012Metric_Pad1.18x1.45mm_HandSolder, F.Cu at (475.5, 258.5)
- added C8: 10uF, Capacitor_SMD:C_0805_2012Metric_Pad1.18x1.45mm_HandSolder, F.Cu at (478.0, 258.5)
- moved R1 5.94 mm to (121.8, 261.0), turned to 0 degrees
- moved R2 5.94 mm to (361.8, 261.0), turned to 0 degrees
- moved R5 5.94 mm to (241.8, 261.0), turned to 0 degrees
- moved R6 5.94 mm to (481.8, 261.0), turned to 0 degrees
Routing:
- net +3.3V: track 393.3 -> 412.0 mm
- net GND: track 484.1 -> 491.0 mm
- net Net-(U3-WAKE/SPI_MOSI): track 8.53 -> 2.59 mm
- net Net-(U2-WAKE/SPI_MOSI): track 8.53 -> 2.61 mm
- net Net-(U1-WAKE/SPI_MOSI): track 8.53 -> 2.61 mm
- net Net-(U4-WAKE/SPI_MOSI): track 8.52 -> 2.61 mm
