File: touch-pads/touch-pads.kicad_pcb (KiCad board)
At the start: 2 copper layers, 500 x 138.2 mm, 63 parts, among them J1 Conn_01x06_Socket, K1 Conn_01x01, K10 Conn_01x01, K11 Conn_01x01, K12 Conn_01x01, K13 Conn_01x01, K14 Conn_01x01, K15 Conn_01x01, K16 Conn_01x01, K17 Conn_01x01, K18 Conn_01x01, K19 Conn_01x01, K2 Conn_01x01, K20 Conn_01x01, K21 Conn_01x01, K22 Conn_01x01, K23 Conn_01x01, K24 Conn_01x01, K25 Conn_01x01, K26 Conn_01x01, K27 Conn_01x01, K28 Conn_01x01, K29 Conn_01x01, K3 Conn_01x01, K30 Conn_01x01, K31 Conn_01x01, K32 Conn_01x01, K4 Conn_01x01, K5 Conn_01x01, K6 Conn_01x01, K7 Conn_01x01, K8 Conn_01x01, K9 Conn_01x01, U1 CAP1188-1-CP-TR, U2 CAP1188-1-CP-TR, U3 CAP1188-1-CP-TR, U4 CAP1188-1-CP-TR

Commit message: mounting holes on schematic
Parts:
- removed REF** (x10): MountingHole_3.2mm_M3, MountingHole:MountingHole_3.2mm_M3
- added H1: MountingHole, MountingHole:MountingHole_3.2mm_M3, F.Cu at (54.8, 132.8)
- added H10: MountingHole, MountingHole:MountingHole_3.2mm_M3, F.Cu at (178.8, 132.8)
- added H2: MountingHole, MountingHole:MountingHole_3.2mm_M3, F.Cu at (54.8, 259.0)
- added H3: MountingHole, MountingHole:MountingHole_3.2mm_M3, F.Cu at (178.8, 259.0)
- added H4: MountingHole, MountingHole:MountingHole_3.2mm_M3, F.Cu at (298.8, 259.0)
- added H5: MountingHole, MountingHole:MountingHole_3.2mm_M3, F.Cu at (418.8, 259.0)
- added H6: MountingHole, MountingHole:MountingHole_3.2mm_M3, F.Cu at (542.8, 259.0)
- added H7: MountingHole, MountingHole:MountingHole_3.2mm_M3, F.Cu at (542.8, 132.8)
- added H8: MountingHole, MountingHole:MountingHole_3.2mm_M3, F.Cu at (418.8, 132.8)
- added H9: MountingHole, MountingHole:MountingHole_3.2mm_M3, F.Cu at (298.8, 132.8)

Commit message: update refs and tracks
Parts:
- moved R2 120.0 mm to (241.8, 261.0)
- moved R4 120.0 mm to (250.5, 253.0)
- moved R5 120.0 mm to (361.8, 261.0)
- moved R7 120.0 mm to (370.5, 253.0)
- moved U3 120.0 mm to (364.2, 256.7)
- moved U2 120.0 mm to (244.3, 256.7)
Connections:
- U2 pad 15: Net-(K24-Pin_1) -> Net-(K16-Pin_1)
- U2 pad 16: Net-(K23-Pin_1) -> Net-(K15-Pin_1)
- U2 pad 17: Net-(K22-Pin_1) -> Net-(K14-Pin_1)
- U2 pad 18: Net-(K21-Pin_1) -> Net-(K13-Pin_1)
- U2 pad 19: Net-(K20-Pin_1) -> Net-(K12-Pin_1)
- U2 pad 20: Net-(K19-Pin_1) -> Net-(K11-Pin_1)
- U2 pad 21: Net-(K18-Pin_1) -> Net-(K10-Pin_1)
- U2 pad 22: Net-(K17-Pin_1) -> Net-(K9-Pin_1)
- U3 pad 15: Net-(K16-Pin_1) -> Net-(K24-Pin_1)
- U3 pad 16: Net-(K15-Pin_1) -> Net-(K23-Pin_1)
- U3 pad 17: Net-(K14-Pin_1) -> Net-(K22-Pin_1)
- U3 pad 18: Net-(K13-Pin_1) -> Net-(K21-Pin_1)
- U3 pad 19: Net-(K12-Pin_1) -> Net-(K20-Pin_1)
- U3 pad 20: Net-(K11-Pin_1) -> Net-(K19-Pin_1)
- U3 pad 21: Net-(K10-Pin_1) -> Net-(K18-Pin_1)
- U3 pad 22: Net-(K9-Pin_1) -> Net-(K17-Pin_1)
Routing:
- net GND: track 491.0 -> 493.6 mm
- net Net-(K11-Pin_1): track 123.9 -> 124.8 mm

Commit message: align between two pcbs
Parts:
- moved H1 9.41 mm to (63.8, 130.0)
- moved H7 9.41 mm to (533.8, 130.0)
- moved H2 9.06 mm to (63.8, 260.0)
- moved H6 9.06 mm to (533.8, 260.0)
- moved H10 5.71 mm to (173.8, 130.0)
- moved H8 5.71 mm to (413.8, 130.0)
- moved H9 5.71 mm to (293.8, 130.0)
- moved H3 5.10 mm to (173.8, 260.0)
- moved H4 5.10 mm to (293.8, 260.0)
- moved H5 5.10 mm to (413.8, 260.0)
Other:
- board size 500 x 138.2 mm -> 480 x 140 mm
Changed lines of the file:
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@@
 	(footprint "MountingHole:MountingHole_3.2mm_M3"
 		(layer "F.Cu")
-		(at 542.75 132.75)
+		(at 533.75 130)
 		(descr "Mounting Hole 3.2mm, no annular, M3")
 		(tags "mounting hole 3.2mm no annular m3")
@@
 			(at 0 -4.2 0)
 			(layer "F.SilkS")
+			(hide yes)
 			(effects
 				(font
@@
 	(footprint "MountingHole:MountingHole_3.2mm_M3"
 		(layer "F.Cu")
-		(at 418.75 132.75)
+		(at 413.75 130)
 		(descr "Mounting Hole 3.2mm, no annular, M3")
 		(tags "mounting hole 3.2mm no annular m3")
@@
 			(at 0 -4.2 0)
 			(layer "F.SilkS")
+			(hide yes)
 			(effects
 				(font
@@
 	(footprint "MountingHole:MountingHole_3.2mm_M3"
 		(layer "F.Cu")
-		(at 298.75 132.75)
+		(at 293.75 130)
 		(descr "Mounting Hole 3.2mm, no annular, M3")
 		(tags "mounting hole 3.2mm no annular m3")
@@
 			(at 0 -4.2 0)
 			(layer "F.SilkS")
+			(hide yes)
 			(effects
 				(font
@@
 	(footprint "MountingHole:MountingHole_3.2mm_M3"
 		(layer "F.Cu")
-		(at 54.75 259)
+		(at 63.75 260)
 		(descr "Mounting Hole 3.2mm, no annular, M3")
 		(tags "mounting hole 3.2mm no annular m3")
@@
 			(at 0 -4.2 0)
 			(layer "F.SilkS")
+			(hide yes)
 			(effects
 				(font
@@
 	(footprint "MountingHole:MountingHole_3.2mm_M3"
 		(layer "F.Cu")
-		(at 178.75 132.75)
+		(at 173.75 130)
 		(descr "Mounting Hole 3.2mm, no annular, M3")
 		(tags "mounting hole 3.2mm no annular m3")
@@
 			(at 0 -4.2 0)
 			(layer "F.SilkS")
+			(hide yes)
 			(effects
 				(font
@@
 	(footprint "MountingHole:MountingHole_3.2mm_M3"
 		(layer "F.Cu")
-		(at 418.75 259)
+		(at 413.75 260)
 		(descr "Mounting Hole 3.2mm, no annular, M3")
 		(tags "mounting hole 3.2mm no annular m3")
@@
 			(at 0 -4.2 0)
 			(layer "F.SilkS")
+			(hide yes)
 			(effects
 				(font
@@
 	(footprint "MountingHole:MountingHole_3.2mm_M3"
 		(layer "F.Cu")
-		(at 178.75 259)
+		(at 173.75 260)
 		(descr "Mounting Hole 3.2mm, no annular, M3")
 		(tags "mounting hole 3.2mm no annular m3")
@@
 			(at 0 -4.2 0)
 			(layer "F.SilkS")
+			(hide yes)
 			(effects
 				(font
@@
 	(footprint "MountingHole:MountingHole_3.2mm_M3"
 		(layer "F.Cu")
-		(at 542.75 259)
+		(at 533.75 260)
 		(descr "Mounting Hole 3.2mm, no annular, M3")
 		(tags "mounting hole 3.2mm no annular m3")
@@
 			(at 0 -4.2 0)
 			(layer "F.SilkS")
+			(hide yes)
 			(effects
 				(font
@@
 	(footprint "MountingHole:MountingHole_3.2mm_M3"
 		(layer "F.Cu")
-		(at 54.75 132.75)
+		(at 63.75 130)
 		(descr "Mounting Hole 3.2mm, no annular, M3")
 		(tags "mounting hole 3.2mm no annular m3")
@@
 			(at 0 -4.2 0)
 			(layer "F.SilkS")
+			(hide yes)
 			(effects
 				(font
@@
 	(footprint "MountingHole:MountingHole_3.2mm_M3"
 		(layer "F.Cu")
-		(at 298.75 259)
+		(at 293.75 260)
 		(descr "Mounting Hole 3.2mm, no annular, M3")
 		(tags "mounting hole 3.2mm no annular m3")
@@
 			(at 0 -4.2 0)
 			(layer "F.SilkS")
+			(hide yes)
 			(effects
 				(font
@@
 	)
 	(gr_line
-		(start 178.75 126)
-		(end 178.75 259.5)
+		(start 178.75 127.25)
+		(end 173.75 127.25)
+		(stroke
+			(width 0.1)
+			(type default)
+		)
+		(layer "Dwgs.User")
+	)
+	(gr_line
+		(start 173.75 125)
+		(end 173.75 265.5)
+		(stroke
+			(width 0.1)
+			(type default)
+		)
+		(layer "Dwgs.User")
+	)
+	(gr_line
+		(start 63.75 125)
+		(end 63.75 273.75)
+		(stroke
+			(width 0.1)
+			(type default)
+		)
+		(layer "Dwgs.User")
+	)
+	(gr_line
+		(start 178.75 125)
+		(end 178.75 265.5)
+		(stroke
+			(width 0.1)
+			(type default)
+		)
+		(layer "Dwgs.User")
+	)
+	(gr_line
+		(start 533.75 122.5)
+		(end 533.75 266.5)
+		(stroke
+			(width 0.1)
+			(type default)
+		)
+		(layer "Dwgs.User")
+	)
+	(gr_line
+		(start 418.75 127.75)
+		(end 413.75 127.75)
+		(stroke
+			(width 0.1)
+			(type default)
+		)
+		(layer "Dwgs.User")
+	)
+	(gr_line
+		(start 298.75 125)
+		(end 298.75 268.25)
+		(stroke
+			(width 0.1)
+			(type default)
+		)
+		(layer "Dwgs.User")
+	)
+	(gr_line
+		(start 298.75 127.25)
+		(end 293.75 127.25)
+		(stroke
+			(width 0.1)
+			(type default)
+		)
+		(layer "Dwgs.User")
+	)
+	(gr_line
+		(start 293.75 124)
+		(end 293.75 265.5)
 		(stroke
 			(width 0.1)
@@
 	)
 	(gr_line
-		(start 542.75 129.75)
-		(end 542.75 260.5)
+		(start 538.75 128.25)
+		(end 533.75 128.25)
 		(stroke
 			(width 0.1)
@@
 	)
 	(gr_line
-		(start 298.75 129)
-		(end 298.75 259.75)
+		(start 413.75 123.25)
+		(end 413.75 266)
 		(stroke
 			(width 0.1)
@@
 	)
 	(gr_line
-		(start 54.75 259)
-		(end 547.5 259)
+		(start 54.75 260)
+		(end 547.5 260)
 		(stroke
 			(width 0.1)
@@
 	)
 	(gr_line
-		(start 54.75 132.75)
-		(end 547.5 132.75)
+		(start 557.5 130)
+		(end 59 130)
 		(stroke
 			(width 0.1)
@@
 	(gr_line
 		(start 418.75 124.25)
-		(end 418.75 259.5)
+		(end 418.75 266.25)
 		(stroke
 			(width 0.1)
@@
 	)
 	(gr_rect
-		(start 48.75 126.75)
-		(end 548.75 265)
+		(start 58.75 125)
+		(end 538.75 265)
 		(stroke
 			(width 0.05)

Commit message: adjust text
Other:
- board text added: "SMCLK SMDATA RESET +3.3V GND ALERT"
Changed lines of the file:
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@@
 		(tags "connector JST XH vertical")
 		(property "Reference" "J1"
-			(at 6.25 3.55 0)
+			(at -4.25 -0.525 0)
 			(unlocked yes)
 			(layer "B.SilkS")
@@
 		(layer "Edge.Cuts")
 	)
+	(gr_text "SMCLK\nSMDATA\nRESET\n+3.3V\nGND\nALERT"
+		(at 270.75 254.75 -90)
+		(layer "B.SilkS")
+		(effects
+			(font
+				(size 1 1)
+				(thickness 0.15)
+			)
+			(justify left bottom mirror)
+		)
+	)
 	(segment
