File: kicad/touch-pads-split/touch-pads.kicad_pcb (KiCad board)
At the start: 2 copper layers, 120 x 140 mm, 19 parts, among them J1 Conn_01x06_Socket, J2 Conn_01x06_Socket, K1 Conn_01x01, K2 Conn_01x01, K3 Conn_01x01, K4 Conn_01x01, K5 Conn_01x01, K6 Conn_01x01, K7 Conn_01x01, K8 Conn_01x01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

Commit message: move common lib, cleanup tracks, logo
Parts:
- added G***: LOGO, Logo:Snep_Copper, B.Cu at (164.5, 256.2)
Routing:
- net Net-(K2-Pin_1): track 91.4 -> 79.4 mm
- net Net-(K4-Pin_1): track 60.9 -> 48.9 mm
