File: kicad/mainboard/mainboard.kicad_pcb (KiCad board)
At the start: 2 copper layers, 40 x 57 mm, 34 parts, among them J1 USB_C_Receptacle_USB2.0_16P, J2 Conn_01x07_Socket, J3 Conn_01x06_Socket, J4 Conn_01x03_Socket, J5 Conn_01x07_Socket, U1 TPD1E05U06DYA, U2 TPD1E05U06DYA, U3 ESP32-S3-WROOM-1, U4 TPD1E05U06DYA, U5 TLV1117-33

Commit message: remove switch lib, add label for led connectors
Other:
- board text added: "+5V GND LED_DATA"
Changed lines of the file:
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@@
 			(net 0)
 			(net_name "")
-			(layers "*.Cu")
+			(layers "F&B.Cu")
 			(name "antenna keepout")
 			(hatch edge 0.508)
@@
 		(tags "capacitor electrolytic")
 		(property "Reference" "C6"
-			(at 4.95 2.25 360)
+			(at 4.95 2.25 0)
 			(layer "F.SilkS")
 			(effects
@@
 		)
 		(property "Value" "100uF"
-			(at 0 4.35 360)
+			(at 0 4.35 0)
 			(layer "F.Fab")
 			(effects
@@
 		)
 		(fp_text user "${REFERENCE}"
-			(at 0 0 360)
+			(at 0 0 0)
 			(layer "F.Fab")
 			(effects
@@
 		)
 	)
+	(gr_text "+5V\nGND\nLED_DATA"
+		(at 115 86.75 0)
+		(layer "F.SilkS")
+		(effects
+			(font
+				(size 0.6 0.6)
+				(thickness 0.1)
+			)
+			(justify left bottom)
+		)
+	)

Commit message: fixup stuff
Connections:
- J4 pad 1: +5V -> LED_DATA
- J4 pad 2: GND -> +5V
- J4 pad 3: LED_DATA -> GND
Routing:
- net LED_DATA: track 12.2 -> 19.5 mm
- net +5V: track 39.8 -> 43.5 mm
- net GND: track 227.1 -> 228.1 mm, vias 6 -> 5
Other:
- board text added: "INT RESET SMDATA SMCLK LPN1 +3.3V GND"
- board text added: "LED_DATA +5V GND"
- board text removed: "+5V GND LED_DATA"
- board text removed: "INT RESET DATA CLK LPN1 +3.3V GND"
Changed lines of the file:
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@@
 		(tags "esp32-s3")
 		(property "Reference" "U3"
-			(at 3.15 11.36 0)
+			(at 0 -17.05 180)
 			(layer "F.SilkS")
 			(effects
@@
 		)
 		(property "Value" "ESP32-S3-WROOM-1"
-			(at 0 12 0)
+			(at 0 12 180)
 			(layer "F.Fab")
 			(effects
@@
 		)
 		(property "Footprint" "PCM_Espressif:ESP32-S3-WROOM-1"
-			(at 0 0 0)
+			(at 0 0 180)
 			(layer "F.Fab")
 			(hide yes)
@@
 		)
 		(property "Datasheet" "https://www.espressif.com/sites/default/files/documentation/esp32-s3-wroom-1_wroom-1u_datasheet_en.pdf"
-			(at 0 0 0)
+			(at 0 0 180)
 			(layer "F.Fab")
 			(hide yes)
@@
 		)
 		(property "Description" "2.4 GHz WiFi (802.11 b/g/n) and Bluetooth ® 5 (LE) module Built around ESP32S3 series of SoCs, Xtensa ® dualcore 32bit LX7 microprocessor Flash up to 16 MB, PSRAM up to 8 MB 36 GPIOs, rich set of peripherals Onboard PCB antenna"
-			(at 0 0 0)
+			(at 0 0 180)
 			(layer "F.Fab")
 			(hide yes)
@@
 		)
 		(fp_text user "Antenna Area"
-			(at 0 -12.75 0)
+			(at 0 -12.75 180)
 			(layer "F.SilkS")
 			(effects
@@
 		)
 		(fp_text user "Antenna Area"
-			(at 0 -12.75 0)
+			(at 0 -12.75 180)
 			(layer "Eco2.User")
 			(effects
@@
 		)
 		(fp_text user "${REFERENCE}"
-			(at 0 0 0)
+			(at 0 0 180)
 			(layer "F.Fab")
 			(effects
@@
 			(size 1 2.1)
 			(drill oval 0.6 1.7)
+			(property pad_prop_heatsink)
 			(layers "*.Cu" "*.Mask" "F.Paste")
 			(remove_unused_layers no)
@@
 			(size 1 1.8)
 			(drill oval 0.6 1.4)
+			(property pad_prop_heatsink)
 			(layers "*.Cu" "*.Mask" "F.Paste")
 			(remove_unused_layers no)
@@
 			(size 1 2.1)
 			(drill oval 0.6 1.7)
+			(property pad_prop_heatsink)
 			(layers "*.Cu" "*.Mask" "F.Paste")
 			(remove_unused_layers no)
@@
 			(size 1 1.8)
 			(drill oval 0.6 1.4)
+			(property pad_prop_heatsink)
 			(layers "*.Cu" "*.Mask" "F.Paste")
 			(remove_unused_layers no)
@@
 			(layers "F.Cu" "F.Paste" "F.Mask")
 			(roundrect_rratio 0.25)
-			(net 4 "+5V")
+			(net 34 "LED_DATA")
 			(pinfunction "Pin_1")
 			(pintype "passive")
@@
 			(layers "F.Cu" "F.Paste" "F.Mask")
 			(roundrect_rratio 0.25)
-			(net 1 "GND")
+			(net 4 "+5V")
 			(pinfunction "Pin_2")
 			(pintype "passive")
@@
 			(layers "F.Cu" "F.Paste" "F.Mask")
 			(roundrect_rratio 0.25)
-			(net 34 "LED_DATA")
+			(net 1 "GND")
 			(pinfunction "Pin_3")
 			(pintype "passive")
@@
 	)
 	(gr_text "SMCLK\nSMDATA\nRESET\n+3.3V\nGND\nALERT"
-		(at 137.5 93.5 0)
+		(at 137.5 92.5 0)
 		(layer "F.SilkS")
 		(effects
@@
 		)
 	)
-	(gr_text "INT\nRESET\nDATA\nCLK\nLPN1\n+3.3V\nGND"
-		(at 110.75 102.5 0)
+	(gr_text "INT\nRESET\nSMDATA\nSMCLK\nLPN1\n+3.3V\nGND"
+		(at 110.75 105.5 0)
 		(layer "F.SilkS")
 		(effects
@@
 	)
 	(gr_text "GND\n+3.3V\nLPN0\nSMCLK\nSMDATA\nRESET\nINT"
-		(at 137.5 106.5 0)
+		(at 137.5 105.5 0)
 		(layer "F.SilkS")
 		(effects
@@
 		)
 	)
-	(gr_text "+5V\nGND\nLED_DATA"
-		(at 115 86.75 0)
+	(gr_text "LED_DATA\n+5V\nGND"
+		(at 115 87 0)
 		(layer "F.SilkS")
 		(effects
@@
 	)
 	(segment
+		(start 110.6 87.75)
+		(end 112.35 87.75)
+		(width 0.6)
+		(layer "F.Cu")
+		(net 1)
+	)
+	(segment
 		(start 121.05 71.68)
 		(end 120.505 71.68)
@@
 	)
 	(segment
-		(start 109.25 84.5)
-		(end 110.5 85.75)
+		(start 109.25 77.8)
+		(end 109.25 86.4)
 		(width 0.6)
 		(layer "F.Cu")
@@
 	)
 	(segment
-		(start 109.25 77.8)
-		(end 109.25 84.5)
-		(width 0.6)
-		(layer "F.Cu")
-		(net 1)
-	)
-	(segment
 		(start 130.9625 82.05)
 		(end 132.75 82.05)
@@
 	)
 	(segment
-		(start 124.25 104)
-		(end 127.05 104)
+		(start 117.25 87.75)
+		(end 112.35 87.75)
 		(width 0.4)
 		(layer "F.Cu")
@@
 	)
 	(segment
-		(start 110.5 85.75)
-		(end 112.35 85.75)
-		(width 0.6)
+		(start 124.25 104)
+		(end 127.05 104)
+		(width 0.4)
 		(layer "F.Cu")
 		(net 1)
@@
 	)
 	(segment
-		(start 115.5 85.75)
-		(end 112.35 85.75)
-		(width 0.4)
-		(layer "F.Cu")
-		(net 1)
-	)
-	(segment
 		(start 130.4 72.935)
 		(end 128.57 71.105)
@@
 	)
 	(segment
+		(start 119 89.5)
+		(end 117.25 87.75)
+		(width 0.4)
+		(layer "F.Cu")
+		(net 1)
+	)
+	(segment
 		(start 140.25 98.75)
 		(end 140.5 98.5)
@@
 	)
 	(segment
+		(start 109.25 86.4)
+		(end 110.6 87.75)
+		(width 0.6)
+		(layer "F.Cu")
+		(net 1)
+	)
+	(segment
 		(start 121.2 74.5)
 		(end 120.7 75)
@@
 		(net 1)
 	)
-	(via
-		(at 115.5 85.75)
-		(size 0.6)
-		(drill 0.3)
-		(layers "F.Cu" "B.Cu")
-		(net 1)
-	)
 	(segment
 		(start 129.5 113.325)
@@
 	(segment
 		(start 119 89.5)
-		(end 119 89.25)
-		(width 0.4)
-		(layer "B.Cu")
-		(net 1)
-	)
-	(segment
-		(start 119 89.25)
-		(end 115.5 85.75)
-		(width 0.4)
-		(layer "B.Cu")
-		(net 1)
-	)
-	(segment
-		(start 119 89.5)
 		(end 119 109.098528)
 		(width 0.4)
@@
 	)
 	(segment
+		(start 115.25 85.75)
+		(end 112.35 85.75)
+		(width 0.6)
+		(layer "F.Cu")
+		(net 4)
+	)
+	(segment
 		(start 129 74.05)
 		(end 129 75.25)
@@
 	)
 	(segment
-		(start 116.7 75.75)
-		(end 112.35 80.1)
-		(width 0.6)
-		(layer "F.Cu")
-		(net 4)
-	)
-	(segment
 		(start 128.35 76.35)
 		(end 123.4 76.35)
@@
 	)
 	(segment
-		(start 126 73.25)
-		(end 128.2 73.25)
+		(start 116.65 75.75)
+		(end 116.65 84.35)
 		(width 0.6)
 		(layer "F.Cu")
@@
 	)
 	(segment
-		(start 116.7 75.75)
-		(end 118.5 75.75)
+		(start 116.65 84.35)
+		(end 115.25 85.75)
 		(width 0.6)
 		(layer "F.Cu")
@@
 	)
 	(segment
-		(start 112.35 80.1)
-		(end 112.35 83.75)
+		(start 126 73.25)
+		(end 128.2 73.25)
+		(width 0.6)
+		(layer "F.Cu")
+		(net 4)
+	)
+	(segment
+		(start 116.7 75.75)
+		(end 118.5 75.75)
 		(width 0.6)
 		(layer "F.Cu")
@@
 	)
 	(segment
-		(start 113.75 89.15)
-		(end 112.35 87.75)
-		(width 0.2)
-		(layer "F.Cu")
-		(net 34)
-	)
-	(segment
-		(start 113.75 90.75)
-		(end 113.75 89.15)
+		(start 115.5 83.75)
+		(end 112.35 83.75)
 		(width 0.2)
 		(layer "F.Cu")
@@
 	)
 	(via
-		(at 113.75 90.75)
+		(at 115.5 83.75)
 		(size 0.6)
 		(drill 0.3)
@@
 	)
 	(segment
-		(start 113.75 90.75)
+		(start 115.5 83.75)
+		(end 113.75 85.5)
+		(width 0.2)
+		(layer "B.Cu")
+		(net 34)
+	)
+	(segment
+		(start 113.75 85.5)
 		(end 113.75 97.65)
 		(width 0.2)
