File: kicad/mainboard/mainboard.kicad_sch (KiCad schematic)
At the start: 28 parts, among them J1 USB_C_Receptacle_USB2.0_16P, J2 Conn_01x03_Socket, J3 Conn_01x06_Socket, J4 Conn_01x06_Socket, U1 TPD1E05U06DYA, U2 TPD1E05U06DYA, U3 ESP32-S3-WROOM-1, U4 TPD1E05U06DYA, U5 TLV1117-33

Commit message: change led to 11
Connections:
- net LED_DATA: now also U3.19 (GPIO11/TOUCH11/ADC2_CH0/FSPID/FSPIIO5/SUBSPID); no longer U3.28 (SPIIO6/GPIO35/FSPID/SUBSPID)
Changed lines of the file:
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@@
-	)
-	(no_connect
-		(at 132.08 173.99)
 	)
 	(no_connect
@@
 	)
 	(no_connect
+		(at 40.64 196.85)
+	)
+	(no_connect
 		(at 132.08 151.13)
 	)
@@
 	(wire
 		(pts
-			(xy 38.1 196.85) (xy 40.64 196.85)
-		)
-		(stroke
-			(width 0)
-			(type default)
-		)
-	)
-	(wire
-		(pts
 			(xy 149.86 143.51) (xy 149.86 144.78)
 		)
@@
 		(pts
 			(xy 134.62 78.74) (xy 134.62 80.01)
+		)
+		(stroke
+			(width 0)
+			(type default)
+		)
+	)
+	(wire
+		(pts
+			(xy 132.08 173.99) (xy 135.89 173.99)
 		)
 		(stroke
@@
 	(global_label "LED_DATA"
 		(shape input)
-		(at 38.1 196.85 180)
+		(at 135.89 173.99 0)
 		(fields_autoplaced yes)
 		(effects
@@
 				(size 1.27 1.27)
 			)
-			(justify right)
+			(justify left)
 		)
 		(property "Intersheetrefs" "${INTERSHEET_REFS}"
-			(at 26.2853 196.85 0)
+			(at 147.7047 173.99 0)
 			(effects
 				(font
 					(size 1.27 1.27)
 				)
-				(justify right)
+				(justify left)
 				(hide yes)
 			)
