File: kicad/touch-pads/touch-pads.kicad_pcb (KiCad board)
At the start: 2 copper layers, 120 x 140 mm, 20 parts, among them J1 Conn_01x06_Socket, J2 Conn_01x06_Socket, K1 Conn_01x01, K2 Conn_01x01, K3 Conn_01x01, K4 Conn_01x01, K5 Conn_01x01, K6 Conn_01x01, K7 Conn_01x01, K8 Conn_01x01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

Commit message: update touch pad
Parts:
- removed H3, H4: MountingHole, MountingHole:MountingHole_3.2mm_M3
- added C10: 0.1uF, Capacitor_SMD:C_0805_2012Metric_Pad1.18x1.45mm_HandSolder, B.Cu at (293.5, 130.0)
- added C11: 0.1uF, Capacitor_SMD:C_0805_2012Metric_Pad1.18x1.45mm_HandSolder, B.Cu at (274.5, 130.0)
- added C12: 0.1uF, Capacitor_SMD:C_0805_2012Metric_Pad1.18x1.45mm_HandSolder, B.Cu at (209.5, 130.0)
- added C13: 0.1uF, Capacitor_SMD:C_0805_2012Metric_Pad1.18x1.45mm_HandSolder, B.Cu at (255.2, 130.0)
- added C14: 0.1uF, Capacitor_SMD:C_0805_2012Metric_Pad1.18x1.45mm_HandSolder, B.Cu at (216.2, 130.0)
- added C3: 0.1uF, Capacitor_SMD:C_0805_2012Metric_Pad1.18x1.45mm_HandSolder, B.Cu at (283.2, 130.0)
- added C4: 0.1uF, Capacitor_SMD:C_0805_2012Metric_Pad1.18x1.45mm_HandSolder, B.Cu at (264.8, 130.0)
- added C5: 0.1uF, Capacitor_SMD:C_0805_2012Metric_Pad1.18x1.45mm_HandSolder, B.Cu at (272.2, 243.8)
- added C6: 10uF, Capacitor_SMD:C_0805_2012Metric_Pad1.18x1.45mm_HandSolder, B.Cu at (269.5, 243.8)
- added C7: 0.1uF, Capacitor_SMD:C_0805_2012Metric_Pad1.18x1.45mm_HandSolder, B.Cu at (245.2, 130.0)
- added C8: 0.1uF, Capacitor_SMD:C_0805_2012Metric_Pad1.18x1.45mm_HandSolder, B.Cu at (235.8, 130.0)
- added C9: 0.1uF, Capacitor_SMD:C_0805_2012Metric_Pad1.18x1.45mm_HandSolder, B.Cu at (226.0, 130.0)
- added D1: WS2812B-4020, WS2812B-4020:WS2812B-4020, F.Cu at (311.5, 131.3)
- added D10: WS2812B-4020, WS2812B-4020:WS2812B-4020, F.Cu at (224.5, 131.3)
- added D11: WS2812B-4020, WS2812B-4020:WS2812B-4020, F.Cu at (215.0, 131.3)
- added D12: WS2812B-4020, WS2812B-4020:WS2812B-4020, F.Cu at (205.2, 131.3)
- added D2: WS2812B-4020, WS2812B-4020:WS2812B-4020, F.Cu at (302.0, 131.3)
- added D3: WS2812B-4020, WS2812B-4020:WS2812B-4020, F.Cu at (292.2, 131.3)
- added D4: WS2812B-4020, WS2812B-4020:WS2812B-4020, F.Cu at (282.5, 131.3)
- added D5: WS2812B-4020, WS2812B-4020:WS2812B-4020, F.Cu at (273.0, 131.3)
- added D6: WS2812B-4020, WS2812B-4020:WS2812B-4020, F.Cu at (263.2, 131.3)
- added D7: WS2812B-4020, WS2812B-4020:WS2812B-4020, F.Cu at (253.5, 131.3)
- added D8: WS2812B-4020, WS2812B-4020:WS2812B-4020, F.Cu at (244.0, 131.3)
- added D9: WS2812B-4020, WS2812B-4020:WS2812B-4020, F.Cu at (234.2, 131.3)
- added J3: Conn_01x03_Socket, Connector_JST:JST_PH_S3B-PH-SM4-TB_1x03-1MP_P2.00mm_Horizontal, B.Cu at (291.0, 117.5)
- added J4: Conn_01x03_Socket, Connector_JST:JST_PH_S3B-PH-SM4-TB_1x03-1MP_P2.00mm_Horizontal, B.Cu at (235.5, 117.5)
- C1, R1, R2, U1: moved to B.Cu
- C2: value 10uF -> 0.1uF; moved to B.Cu
- moved C2 233.7 mm to (313.0, 130.0), turned to 90 degrees
- moved C1 227.7 mm to (303.2, 130.0), turned to 90 degrees
- moved H1 153.3 mm to (215.2, 106.8)
- moved J1 149.8 mm to (238.5, 252.0)
- moved G*** 149.5 mm to (314.0, 255.0)
- moved K1 146.1 mm to (219.8, 158.2)
- moved K2 146.1 mm to (219.8, 212.2)
- moved K3 145.1 mm to (248.8, 158.2)
- moved K4 145.1 mm to (248.8, 212.2)
- moved R1 144.8 mm to (265.8, 245.8), turned to 180 degrees
- moved K5 144.1 mm to (277.8, 158.2)
- moved K6 144.1 mm to (277.8, 212.2)
- moved K7 143.1 mm to (306.8, 158.2)
- moved K8 143.1 mm to (306.8, 212.2)
- moved U1 139.9 mm to (263.2, 241.0)
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Connections:
- C1 pad 1: +3.3V -> GND
- C1 pad 2: GND -> +5V
- C2 pad 1: +3.3V -> GND
- C2 pad 2: GND -> +5V
Routing:
- net GND: track 84.6 -> 295.8 mm, vias 1 -> 14
- net +5V: track 0.00 -> 202.7 mm, vias 0 -> 12
- net LED_DATA_OUT: track 0.00 -> 41.6 mm, vias 0 -> 1
- net LED_DATA_IN: track 0.00 -> 31.6 mm, vias 0 -> 1
- net Net-(D2-DOUT): track 0.00 -> 15.4 mm
- net Net-(D6-DOUT): track 0.00 -> 15.4 mm
- net Net-(D8-DOUT): track 0.00 -> 15.4 mm
- net Net-(D4-DOUT): track 0.00 -> 15.1 mm
- net Net-(D10-DOUT): track 0.00 -> 14.9 mm
- net Net-(D7-DOUT): track 0.00 -> 14.5 mm
- net Net-(D5-DOUT): track 0.00 -> 14.4 mm
- net Net-(D10-DIN): track 0.00 -> 14.3 mm
- net Net-(D11-DOUT): track 0.00 -> 14.2 mm
- net Net-(D3-DOUT): track 0.00 -> 14.2 mm
- net Net-(D1-DOUT): track 0.00 -> 14.2 mm
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Other:
- board size 120 x 140 mm -> 119.5 x 161 mm
- board text added: "GND +5V LED_DATA_IN"
- board text added: "GND +5V LED_DATA_OUT"

Commit message: fix some 3d models
Parts:
- D1, D10, D11, D12, D2, D3, D4, D5, D6, D7, D8, D9: value WS2812B-4020 -> LED_WS2812B-4020
Changed lines of the file:
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@@
 			)
 		)
-		(property "Value" "WS2812B-4020"
+		(property "Value" "LED_WS2812B-4020"
 			(at 7.92 3.185 0)
 			(layer "F.Fab")
@@
 			(solder_mask_margin 0.102)
 		)
-		(model "${KIPRJMOD}/lib/WS2812B-4020/WS2812B-4020.step"
+		(model "${KIPRJMOD}/../lib/WS2812B-4020/WS2812B-4020.step"
 			(offset
 				(xyz 0 -1 1)
@@
 			)
 		)
-		(property "Value" "WS2812B-4020"
+		(property "Value" "LED_WS2812B-4020"
 			(at 7.92 3.185 0)
 			(layer "F.Fab")
@@
 			(solder_mask_margin 0.102)
 		)
-		(model "${KIPRJMOD}/lib/WS2812B-4020/WS2812B-4020.step"
+		(model "${KIPRJMOD}/../lib/WS2812B-4020/WS2812B-4020.step"
 			(offset
 				(xyz 0 -1 1)
@@
 			)
 		)
-		(property "Value" "WS2812B-4020"
+		(property "Value" "LED_WS2812B-4020"
 			(at 7.92 3.185 0)
 			(layer "F.Fab")
@@
 			(solder_mask_margin 0.102)
 		)
-		(model "${KIPRJMOD}/lib/WS2812B-4020/WS2812B-4020.step"
+		(model "${KIPRJMOD}/../lib/WS2812B-4020/WS2812B-4020.step"
 			(offset
 				(xyz 0 -1 1)
@@
 			)
 		)
-		(property "Value" "WS2812B-4020"
+		(property "Value" "LED_WS2812B-4020"
 			(at 7.92 3.185 0)
 			(layer "F.Fab")
@@
 			(solder_mask_margin 0.102)
 		)
-		(model "${KIPRJMOD}/lib/WS2812B-4020/WS2812B-4020.step"
+		(model "${KIPRJMOD}/../lib/WS2812B-4020/WS2812B-4020.step"
 			(offset
 				(xyz 0 -1 1)
@@
 			)
 		)
-		(property "Value" "WS2812B-4020"
+		(property "Value" "LED_WS2812B-4020"
 			(at 7.92 3.185 0)
 			(layer "F.Fab")
@@
 			(solder_mask_margin 0.102)
 		)
-		(model "${KIPRJMOD}/lib/WS2812B-4020/WS2812B-4020.step"
+		(model "${KIPRJMOD}/../lib/WS2812B-4020/WS2812B-4020.step"
 			(offset
 				(xyz 0 -1 1)
@@
 			)
 		)
-		(property "Value" "WS2812B-4020"
+		(property "Value" "LED_WS2812B-4020"
 			(at 7.92 3.185 0)
 			(layer "F.Fab")
@@
 			(solder_mask_margin 0.102)
 		)
-		(model "${KIPRJMOD}/lib/WS2812B-4020/WS2812B-4020.step"
+		(model "${KIPRJMOD}/../lib/WS2812B-4020/WS2812B-4020.step"
 			(offset
 				(xyz 0 -1 1)
@@
 			)
 		)
-		(property "Value" "WS2812B-4020"
+		(property "Value" "LED_WS2812B-4020"
 			(at 7.92 3.185 0)
 			(layer "F.Fab")
@@
 			(solder_mask_margin 0.102)
 		)
-		(model "${KIPRJMOD}/lib/WS2812B-4020/WS2812B-4020.step"
+		(model "${KIPRJMOD}/../lib/WS2812B-4020/WS2812B-4020.step"
 			(offset
 				(xyz 0 -1 1)
@@
 			)
 		)
-		(property "Value" "WS2812B-4020"
+		(property "Value" "LED_WS2812B-4020"
 			(at 7.92 3.185 0)
 			(layer "F.Fab")
@@
 			(solder_mask_margin 0.102)
 		)
-		(model "${KIPRJMOD}/lib/WS2812B-4020/WS2812B-4020.step"
+		(model "${KIPRJMOD}/../lib/WS2812B-4020/WS2812B-4020.step"
 			(offset
 				(xyz 0 -1 1)
@@
 			)
 		)
-		(property "Value" "WS2812B-4020"
+		(property "Value" "LED_WS2812B-4020"
 			(at 7.92 3.185 0)
 			(layer "F.Fab")
@@
 			(solder_mask_margin 0.102)
 		)
-		(model "${KIPRJMOD}/lib/WS2812B-4020/WS2812B-4020.step"
+		(model "${KIPRJMOD}/../lib/WS2812B-4020/WS2812B-4020.step"
 			(offset
 				(xyz 0 -1 1)
@@
 			)
 		)
-		(property "Value" "WS2812B-4020"
+		(property "Value" "LED_WS2812B-4020"
 			(at 7.92 3.185 0)
 			(layer "F.Fab")
@@
 			(solder_mask_margin 0.102)
 		)
-		(model "${KIPRJMOD}/lib/WS2812B-4020/WS2812B-4020.step"
+		(model "${KIPRJMOD}/../lib/WS2812B-4020/WS2812B-4020.step"
 			(offset
 				(xyz 0 -1 1)
@@
 			)
 		)
-		(property "Value" "WS2812B-4020"
+		(property "Value" "LED_WS2812B-4020"
 			(at 7.92 3.185 0)
 			(layer "F.Fab")
@@
 			(solder_mask_margin 0.102)
 		)
-		(model "${KIPRJMOD}/lib/WS2812B-4020/WS2812B-4020.step"
+		(model "${KIPRJMOD}/../lib/WS2812B-4020/WS2812B-4020.step"
 			(offset
 				(xyz 0 -1 1)
@@
 			)
 		)
-		(property "Value" "WS2812B-4020"
+		(property "Value" "LED_WS2812B-4020"
 			(at 7.92 3.185 0)
 			(layer "F.Fab")
@@
 			(solder_mask_margin 0.102)
 		)
-		(model "${KIPRJMOD}/lib/WS2812B-4020/WS2812B-4020.step"
+		(model "${KIPRJMOD}/../lib/WS2812B-4020/WS2812B-4020.step"
 			(offset
 				(xyz 0 -1 1)
@@
 		)
 		(fp_text user "*"
-			(at -3.0099 1.524 90)
+			(at -3.0099 1.524 -90)
 			(layer "B.SilkS")
 			(effects
@@
 		)
 		(fp_text user "*"
-			(at -3.0099 1.524 90)
+			(at -3.0099 1.524 -90)
 			(layer "B.SilkS")
 			(effects
@@
 			)
 		)
-		(fp_text user "*"
-			(at -1.5621 1.524 -90)
+		(fp_text user "${REFERENCE}"
+			(at 0 0 -90)
 			(unlocked yes)
 			(layer "B.Fab")
@@
 			)
 		)
-		(fp_text user "${REFERENCE}"
-			(at 0 0 -90)
+		(fp_text user "*"
+			(at -1.5621 1.524 -90)
 			(unlocked yes)
 			(layer "B.Fab")
@@
 			(pintype "passive")
 		)
-		(model "${KIPRJMOD}/lib/CAP1188_1_CP_TR/QFN24_4X4MC_MCH.step"
+		(model "${KIPRJMOD}/../lib/CAP1188_1_CP_TR/QFN24_4X4MC_MCH.step"
 			(offset
 				(xyz 0 0 0)
@@
 		(tags "connector JST GH horizontal")
 		(property "Reference" "J1"
-			(at 7 0 360)
+			(at 7 0 0)
 			(layer "B.SilkS")
 			(effects
@@
 		(tags "connector JST GH horizontal")
 		(property "Reference" "J2"
-			(at -7 0 360)
+			(at -7 0 0)
 			(layer "B.SilkS")
 			(effects

Commit message: fixup stuff
Routing:
- net Net-(K1-Pin_1): track 143.2 -> 144.0 mm
Changed lines of the file:
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@@
 		(pad "1" smd roundrect
 			(at 0 -3.25)
-			(size 26.5 45.5)
+			(size 27 45.5)
 			(layers "F.Cu")
 			(roundrect_rratio 0.01923076923)
@@
 		(pad "1" smd roundrect
 			(at 0 -3.25 180)
-			(size 26.5 45.5)
+			(size 27 45.5)
 			(layers "F.Cu")
 			(roundrect_rratio 0.01923076923)
@@
 		(pad "1" smd roundrect
 			(at 0 -3.25)
-			(size 26.5 45.5)
+			(size 27 45.5)
 			(layers "F.Cu")
 			(roundrect_rratio 0.01923076923)
@@
 		(pad "1" smd roundrect
 			(at 0 -3.25 180)
-			(size 26.5 45.5)
+			(size 27 45.5)
 			(layers "F.Cu")
 			(roundrect_rratio 0.01923076923)
@@
 		(pad "1" smd roundrect
 			(at 0 -3.25)
-			(size 26.5 45.5)
+			(size 27 45.5)
 			(layers "F.Cu")
 			(roundrect_rratio 0.01923076923)
@@
 		(pad "1" smd roundrect
 			(at 0 -3.25)
-			(size 26.5 45.5)
+			(size 27 45.5)
 			(layers "F.Cu")
 			(roundrect_rratio 0.01923076923)
@@
 		(pad "1" smd roundrect
 			(at 0 -3.25 180)
-			(size 26.5 45.5)
+			(size 27 45.5)
 			(layers "F.Cu")
 			(roundrect_rratio 0.01923076923)
@@
 		(pad "1" smd roundrect
 			(at 0 -3.25 180)
-			(size 26.5 45.5)
+			(size 27 45.5)
 			(layers "F.Cu")
 			(roundrect_rratio 0.01923076923)
@@
 			)
 		)
-		(fp_text user "${REFERENCE}"
-			(at 0 0 -90)
+		(fp_text user "*"
+			(at -1.5621 1.524 -90)
 			(unlocked yes)
 			(layer "B.Fab")
@@
 			)
 		)
-		(fp_text user "*"
-			(at -1.5621 1.524 -90)
+		(fp_text user "${REFERENCE}"
+			(at 0 0 -90)
 			(unlocked yes)
 			(layer "B.Fab")
@@
 	)
 	(segment
-		(start 206.2 232.45)
-		(end 206.2 175.05)
-		(width 0.2)
-		(layer "F.Cu")
-		(net 7)
-	)
-	(segment
-		(start 267 241.75)
-		(end 266.5 241.25)
+		(start 205.95 233.2)
+		(end 214.5 241.75)
 		(width 0.2)
 		(layer "F.Cu")
@@
 	)
 	(segment
-		(start 266.5 241.25)
-		(end 215 241.25)
+		(start 205.95 175.3)
+		(end 205.95 233.2)
 		(width 0.2)
 		(layer "F.Cu")
@@
 	)
 	(segment
-		(start 206.2 175.05)
-		(end 219.75 161.5)
+		(start 219.75 161.5)
+		(end 205.95 175.3)
 		(width 0.2)
 		(layer "F.Cu")
@@
 	)
 	(segment
-		(start 215 241.25)
-		(end 206.2 232.45)
+		(start 214.5 241.75)
+		(end 267 241.75)
 		(width 0.2)
 		(layer "F.Cu")

Commit message: touch-pad gerber
Parts:
- D1, D10, D11, D12, D2, D3, D4, D5, D6, D7, D8, D9: value LED_WS2812B-4020 -> WS2812B-4020
Changed lines of the file:
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@@
 			)
 		)
-		(property "Value" "LED_WS2812B-4020"
+		(property "Value" "WS2812B-4020"
 			(at 7.92 3.185 0)
 			(layer "F.Fab")
@@
 			)
 		)
-		(property "Value" "LED_WS2812B-4020"
+		(property "Value" "WS2812B-4020"
 			(at 7.92 3.185 0)
 			(layer "F.Fab")
@@
 			)
 		)
-		(property "Value" "LED_WS2812B-4020"
+		(property "Value" "WS2812B-4020"
 			(at 7.92 3.185 0)
 			(layer "F.Fab")
@@
 			)
 		)
-		(property "Value" "LED_WS2812B-4020"
+		(property "Value" "WS2812B-4020"
 			(at 7.92 3.185 0)
 			(layer "F.Fab")
@@
 			)
 		)
-		(property "Value" "LED_WS2812B-4020"
+		(property "Value" "WS2812B-4020"
 			(at 7.92 3.185 0)
 			(layer "F.Fab")
@@
 			)
 		)
-		(property "Value" "LED_WS2812B-4020"
+		(property "Value" "WS2812B-4020"
 			(at 7.92 3.185 0)
 			(layer "F.Fab")
@@
 			)
 		)
-		(property "Value" "LED_WS2812B-4020"
+		(property "Value" "WS2812B-4020"
 			(at 7.92 3.185 0)
 			(layer "F.Fab")
@@
 			)
 		)
-		(property "Value" "LED_WS2812B-4020"
+		(property "Value" "WS2812B-4020"
 			(at 7.92 3.185 0)
 			(layer "F.Fab")
@@
 			)
 		)
-		(property "Value" "LED_WS2812B-4020"
+		(property "Value" "WS2812B-4020"
 			(at 7.92 3.185 0)
 			(layer "F.Fab")
@@
 			)
 		)
-		(property "Value" "LED_WS2812B-4020"
+		(property "Value" "WS2812B-4020"
 			(at 7.92 3.185 0)
 			(layer "F.Fab")
@@
 			)
 		)
-		(property "Value" "LED_WS2812B-4020"
+		(property "Value" "WS2812B-4020"
 			(at 7.92 3.185 0)
 			(layer "F.Fab")
@@
 			)
 		)
-		(property "Value" "LED_WS2812B-4020"
+		(property "Value" "WS2812B-4020"
 			(at 7.92 3.185 0)
 			(layer "F.Fab")

Commit message: v3 touchpads with Tof sensors
Parts:
- added B1: ~, VL53L5CX_Breakout:VL53L5CX_Breakout_Aliexpress, F.Cu at (265.0, 255.2)
- added J5: Conn_01x06_Socket, Connector_JST:JST_GH_SM06B-GHS-TB_1x06-1MP_P1.25mm_Horizontal, B.Cu at (237.8, 255.0)
- added J6: Conn_01x06_Socket, Connector_JST:JST_GH_SM06B-GHS-TB_1x06-1MP_P1.25mm_Horizontal, B.Cu at (238.2, 239.9)
- added JP1: SolderJumper_2_Open, Jumper:SolderJumper-2_P1.3mm_Open_RoundedPad1.0x1.5mm, B.Cu at (247.6, 254.2)
- added JP2: SolderJumper_2_Open, Jumper:SolderJumper-2_P1.3mm_Open_RoundedPad1.0x1.5mm, B.Cu at (247.6, 251.5)
- added JP3: SolderJumper_2_Open, Jumper:SolderJumper-2_P1.3mm_Open_RoundedPad1.0x1.5mm, B.Cu at (247.6, 248.8)
- added JP4: SolderJumper_2_Open, Jumper:SolderJumper-2_P1.3mm_Open_RoundedPad1.0x1.5mm, B.Cu at (247.6, 246.0)
- C2: value 0.1uF -> 10uF
- C6: value 10uF -> 0.1uF
- J1: value Conn_01x06_Socket -> Conn_01x03_Socket; footprint Connector_JST:JST_GH_SM06B-GHS-TB_1x06-1MP_P1.25mm_Horizontal -> Connector_JST:JST_PH_S3B-PH-SM4-TB_1x03-1MP_P2.00mm_Horizontal
- J3: value Conn_01x03_Socket -> Conn_01x06_Socket; footprint Connector_JST:JST_PH_S3B-PH-SM4-TB_1x03-1MP_P2.00mm_Horizontal -> Connector_JST:JST_GH_SM06B-GHS-TB_1x06-1MP_P1.25mm_Horizontal
- moved J1 144.4 mm to (291.1, 117.5), turned to -90 degrees
- moved J3 137.5 mm to (291.2, 255.0)
- moved C5 122.8 mm to (226.0, 130.0), turned to 90 degrees
- moved C2 120.8 mm to (272.2, 243.8), turned to -90 degrees
- moved C6 118.7 mm to (235.5, 130.0), turned to 90 degrees
- moved C1 118.7 mm to (269.5, 243.8), turned to -90 degrees
- moved C14 96.8 mm to (313.0, 130.0)
- moved C12 84.0 mm to (293.5, 130.0)
- moved C3 73.8 mm to (209.5, 130.0)
- moved C4 48.5 mm to (216.2, 130.0)
- moved C13 48.0 mm to (303.2, 130.0)
- moved C9 38.5 mm to (264.5, 130.0)
- moved C8 19.2 mm to (255.0, 130.0)
- moved C10 19.0 mm to (274.5, 130.0)
- moved J2 12.4 mm to (290.6, 239.9)
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Connections:
- C1 pad 1: GND -> +3.3V
- C1 pad 2: +5V -> GND
- C2 pad 1: GND -> +3.3V
- C2 pad 2: +5V -> GND
- C5 pad 1: +3.3V -> GND
- C5 pad 2: GND -> +5V
- C6 pad 1: +3.3V -> GND
- C6 pad 2: GND -> +5V
- J1 pad 1: SMCLK -> GND
- J1 pad 2: SMDATA -> +5V
- J1 pad 3: RESET -> LED_DATA_IN
- J2 pad 1: ALERT -> TOUCH_ALERT
- J2 pad 2: GND -> TOUCH_RESET
- J2 pad 3: +3.3V -> SMDATA
- J2 pad 4: RESET -> SMCLK
- J2 pad 5: SMDATA -> +3.3V
- J2 pad 6: SMCLK -> GND
- J3 pad 1: GND -> TOF_LPN0
- J3 pad 2: +5V -> TOF_LPN1
- J3 pad 3: LED_DATA_IN -> TOF_LPN2
- U1 pad 13: ALERT -> TOUCH_ALERT
- U1 pad 24: RESET -> TOUCH_RESET
Routing:
- net TOF_LPN3: track 0.00 -> 79.4 mm
- net TOF_LPN2: track 0.00 -> 77.5 mm
- net TOF_LPN1: track 0.00 -> 76.9 mm
- net ALERT: track 73.4 -> 0.00 mm, vias 2 -> 0
- net RESET: track 64.1 -> 0.00 mm, vias 2 -> 0
- net TOUCH_ALERT: track 0.00 -> 63.5 mm
- net TOF_LPN0: track 0.00 -> 58.5 mm
- net TOF_INT: track 0.00 -> 58.3 mm, vias 0 -> 1
- net TOUCH_RESET: track 0.00 -> 56.3 mm, vias 0 -> 2
- net TOF_RESET: track 0.00 -> 49.9 mm
- net Net-(B1-LPN): track 0.00 -> 33.9 mm
- net GND: track 295.8 -> 302.8 mm
- net +3.3V: track 65.6 -> 72.7 mm, vias 2 -> 3
- net SMDATA: track 57.1 -> 63.9 mm, vias 2 -> 1
- net SMCLK: track 58.6 -> 64.7 mm
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
Commit message: cleanup some
Parts:
- moved J3 2.65 mm to (288.6, 255.0)
- moved J2 2.00 mm to (288.6, 239.9)
- moved B1 1.75 mm to (263.2, 255.2)
- moved J6 0.40 mm to (237.8, 239.9)
- moved R2 0.25 mm to (258.8, 238.0)
Routing:
- net SMCLK: track 64.7 -> 62.1 mm
- net Net-(B1-LPN): track 33.9 -> 31.7 mm
- net TOF_INT: track 58.3 -> 56.2 mm
- net TOF_LPN2: track 77.5 -> 75.4 mm
- net TOF_RESET: track 49.9 -> 47.8 mm
- net TOF_LPN3: track 79.4 -> 77.3 mm
- net TOF_LPN1: track 76.9 -> 74.7 mm
- net TOF_LPN0: track 58.5 -> 56.3 mm
- net TOUCH_ALERT: track 63.5 -> 61.7 mm
- net TOUCH_RESET: track 56.3 -> 54.6 mm
- net GND: track 302.8 -> 301.5 mm
- net SMDATA: track 63.9 -> 62.5 mm
Other:
- board text added: "LPN3 LPN2 LPN1 LPN0"
- board text added: "TOF_LPN0 TOF_LPN1 TOF_LPN2 TOF_LPN3 TOF_INT TOF_RESET"
- board text added: "TOUCH_ALERT TOUCH_RESET SMDATA SMCLK +3.3V GND"
- board text removed: "ALERT GND +3.3V RESET SMDATA SMCLK"

Commit message: fixes
Parts:
- moved J2 50.9 mm to (237.8, 239.9), turned to 90 degrees
- moved J3 50.9 mm to (237.8, 255.0), turned to 90 degrees
- moved J5 50.9 mm to (288.6, 255.0), turned to -90 degrees
- moved J6 50.9 mm to (288.6, 239.9), turned to -90 degrees
- moved JP4 8.75 mm to (247.7, 254.8)
- moved JP1 7.75 mm to (247.7, 246.5)
- moved JP3 3.25 mm to (247.7, 252.0)
- moved JP2 2.25 mm to (247.7, 249.2)
- moved R2 1.03 mm to (259.0, 237.0), turned to 180 degrees
Routing:
- net TOF_LPN0: track 56.3 -> 78.9 mm
- net TOUCH_RESET: track 54.6 -> 61.7 mm
- net TOF_LPN2: track 75.4 -> 80.6 mm
- net TOUCH_ALERT: track 61.7 -> 66.9 mm, vias 0 -> 2
- net TOF_LPN1: track 74.7 -> 78.8 mm
- net TOF_RESET: track 47.8 -> 51.4 mm
- net GND: track 301.5 -> 305.0 mm, vias 14 -> 13
- net TOF_LPN3: track 77.3 -> 80.5 mm
- net Net-(U1-ADDR_COMM): track 5.22 -> 3.97 mm
- net +3.3V: track 72.3 -> 73.5 mm
- net SMCLK: track 62.1 -> 63.0 mm
- net TOF_INT: track 56.2 -> 57.1 mm
- net Net-(B1-LPN): track 31.7 -> 32.6 mm
- net SMDATA: track 62.5 -> 62.8 mm, vias 1 -> 2
Other:
- board text added: "GND +3.3V SMCLK SMDATA TOUCH_RESET TOUCH_ALERT"
- board text added: "LPN0 LPN1 LPN2 LPN3"
- board text added: "TOF_RESET TOF_INT TOF_LPN3 TOF_LPN2 TOF_LPN1 TOF_LPN0"
- board text removed: "LPN3 LPN2 LPN1 LPN0"
- board text removed: "TOF_LPN0 TOF_LPN1 TOF_LPN2 TOF_LPN3 TOF_INT TOF_RESET"
- board text removed: "TOUCH_ALERT TOUCH_RESET SMDATA SMCLK +3.3V GND"
